Commit message: correct frame name

File: urdf/cello_description.urdf (robot description, URDF)
Before this commit: robot cello_description, 10 links, 9 joints
Links:
- removed link world
- added link leader_frame

File: urdf/fr3.urdf (robot description, URDF)
Before this commit: robot fr3, 10 links, 9 joints
Links:
- removed link base
- added link fr3_frame

Commit message: Add RViz config and embed meshes; ignore browse db

File: urdf/cello_description.urdf (robot description, URDF)
Before this commit: robot cello_description, 10 links, 9 joints
Links:
- link base_link: geometry collision mesh filename=package://leader_arm_viz/meshes/base_link.STL; visual mesh filename=package://leader_arm_viz/meshes/base_link.STL
- link link1: geometry collision mesh filename=package://leader_arm_viz/meshes/link1.STL; visual mesh filename=package://leader_arm_viz/meshes/link1.STL
- link link2: geometry collision mesh filename=package://leader_arm_viz/meshes/link2.STL; visual mesh filename=package://leader_arm_viz/meshes/link2.STL
- link link3: geometry collision mesh filename=package://leader_arm_viz/meshes/link3.STL; visual mesh filename=package://leader_arm_viz/meshes/link3.STL
- link link4: geometry collision mesh filename=package://leader_arm_viz/meshes/link4.STL; visual mesh filename=package://leader_arm_viz/meshes/link4.STL
- link link5: geometry collision mesh filename=package://leader_arm_viz/meshes/link5.STL; visual mesh filename=package://leader_arm_viz/meshes/link5.STL
- link link6: geometry collision mesh filename=package://leader_arm_viz/meshes/link6.STL; visual mesh filename=package://leader_arm_viz/meshes/link6.STL
- link link7_left: geometry collision mesh filename=package://leader_arm_viz/meshes/link7_left.STL; visual mesh filename=package://leader_arm_viz/meshes/link7_left.STL
- link link7_right: geometry collision mesh filename=package://leader_arm_viz/meshes/link7_right.STL; visual mesh filename=package://leader_arm_viz/meshes/link7_right.STL

Commit message: updated cello urdf to match franka eef frame

File: urdf/cello_description.urdf (robot description, URDF)
Before this commit: robot cello_description, 10 links, 9 joints
Joints:
- joint joint6: origin xyz=-0.00132500000000002 -0.170658355416465 0 rpy=1.5707963267949 -1.5707963267949 0 -> xyz=-0.00132500000000002 -0.170658355416465 0 rpy=1.5707963267949 0 0

Commit message: setting up repo for ros2 in isaacsim

File: urdf/cello_description.urdf (robot description, URDF)
Before this commit: robot cello_description, 10 links, 9 joints
Joints:
- joint joint6: origin xyz=-0.00132500000000002 -0.170658355416465 0 rpy=1.5707963267949 0 0 -> xyz=-0.00132500000000002 -0.170658355416465 0 rpy=1.5707963267949 -1.5707963267949 0
